Commit message: nav2 succeed

File: src/yahboomcar_description/urdf/yahboomcar_R2.urdf (robot description, URDF)
Before this commit: robot yahboomcar, 9 links, 8 joints
Links:
- removed link camera_link
Joints:
- removed joint camera_joint
- joint back_left_joint: origin xyz=-0.11607 0.08425 0.0125 rpy=0 0 0 -> xyz=0.0935 -0.0915 0.02 rpy=0 0 0
- joint back_right_joint: origin xyz=-0.11607 -0.08425 0.0125 rpy=0 0 0 -> xyz=-0.0935 -0.0915 0.02 rpy=0 0 0
- joint front_left_steer_joint: origin xyz=0.11922 0.065 0.0262 rpy=0 0 0 -> xyz=0.0935 0.0915 0.02 rpy=0 0 0
- joint front_right_steer_joint: origin xyz=0.11922 -0.065 0.0242 rpy=0 0 0 -> xyz=0.0935 -0.0915 0.02 rpy=0 0 0
- joint laser_joint: origin xyz=0.012548 0 0.1311 rpy=0 0 0 -> xyz=0 0.0065 0.155 rpy=0 0 0

File: src/yahboomcar_description/yahboomcar_description/urdf/yahboomcar_R2.urdf (robot description, URDF)
Before this commit: robot yahboomcar, 9 links, 8 joints
Links:
- removed link camera_link
- link laser_link: geometry collision mesh filename=package://yahboomcar_description/meshes/laser_link_R2.STL; visual mesh filename=package://yahboomcar_description/meshes/laser_link_R2.STL
Joints:
- removed joint camera_joint
- joint back_left_joint: origin xyz=-0.11607 0.08425 0.0125 rpy=0 0 0 -> xyz=0.0935 -0.0915 0.02 rpy=0 0 0
- joint back_right_joint: origin xyz=-0.11607 -0.08425 0.0125 rpy=0 0 0 -> xyz=-0.0935 -0.0915 0.02 rpy=0 0 0
- joint front_left_steer_joint: origin xyz=0.11922 0.065 0.0262 rpy=0 0 0 -> xyz=0.0935 0.0915 0.02 rpy=0 0 0
- joint front_right_steer_joint: origin xyz=0.11922 -0.065 0.0242 rpy=0 0 0 -> xyz=0.0935 -0.0915 0.02 rpy=0 0 0
- joint laser_joint: origin xyz=0.012548 0 0.1311 rpy=0 0 0 -> xyz=0 0.0065 0.155 rpy=0 0 0

Commit message: 0718

File: src/yahboomcar_description/urdf/yahboomcar_R2.urdf (robot description, URDF)
Before this commit: robot yahboomcar, 8 links, 7 joints
Links:
- removed link laser_link
- added link laser, mass 0; collision mesh filename=package://yahboomcar_description/meshes/laser_link_R2.STL; visual mesh filename=package://yahboomcar_description/meshes/laser_link_R2.STL
Joints:
- joint laser_joint: child laser_link -> laser; origin xyz=0 0.0065 0.155 rpy=0 0 0 -> xyz=0.0 0.0065 0.155 rpy=0 0 3.14159

File: src/yahboomcar_description/yahboomcar_description/urdf/yahboomcar_R2.urdf (robot description, URDF)
Before this commit: robot yahboomcar, 8 links, 7 joints
Links:
- removed link laser_link
- added link laser, mass 0; collision mesh filename=package://yahboomcar_description/meshes/laser_link_R2.STL; visual mesh filename=package://yahboomcar_description/meshes/laser_link_R2.STL
Joints:
- joint laser_joint: child laser_link -> laser
